Commit message: fixed slider (for the boxes to not be moving) & three views to combine

File: toolbox/toolbox.urdf (robot description, URDF)
Before this commit: robot toolbox, 19 links, 18 joints
Joints:
- joint ld1-slider: origin xyz=0.12500000000000011102 0 0.025000000000000077716 rpy=-1.570796326794896558 -2.6469779601696862086e-23 -1.570796326794896558 -> xyz=-0.15 0 0.025000000000000077716 rpy=-1.570796326794896558 -2.6469779601696862086e-23 -1.570796326794896558; type prismatic -> fixed
- joint ld2-slider: type prismatic -> fixed
- joint ld3-slider: type prismatic -> fixed
- joint sd1-slider: type prismatic -> fixed
- joint sd2-slider: type prismatic -> fixed
- joint sd3-slider: type prismatic -> fixed

Commit message: idk wtf honestly

File: toolbox/toolbox.urdf (robot description, URDF)
Before this commit: robot toolbox, 19 links, 18 joints
Links:
- removed link body
- added link body_, mass 152.97898221658957141; collision mesh filename=body.obj; visual mesh filename=body.obj
Joints:
- joint l hinge body fasten: parent body -> body_
- joint ld1-slider: parent body -> body_
- joint ld2-slider: parent body -> body_
- joint ld3-slider: parent body -> body_
- joint r hinge body fasten: parent body -> body_
- joint sd1-slider: parent body -> body_
- joint sd2-slider: parent body -> body_
- joint sd3-slider: parent body -> body_
